Commit message: added camera frame

File: mycobot_320_description/urdf/mycobot_320_macro.xacro (robot description, xacro)
@@ -211,4 +211,11 @@
       <child link="${prefix}tool0"/>
     </joint>
+    <!-- Camera frame -->
+    <link name="${prefix}camera"/>
+    <joint name="${prefix}link6-camera" type="fixed">
+      <origin xyz="0 0 0.075" rpy="0 0 0"/>
+      <parent link="${prefix}link6"/>
+      <child link="${prefix}camera"/>
+    </joint>
   </xacro:macro>
 </robot>

Commit message: added gripper frame

File: mycobot_320_description/urdf/mycobot_320_macro.xacro (robot description, xacro)
@@ -211,4 +211,11 @@
       <child link="${prefix}tool0"/>
     </joint>
+    <!-- Gripper -->
+    <link name="${prefix}gripper"/>
+    <joint name="${prefix}link6-gripper" type="fixed">
+      <origin xyz="0 0 0.025" rpy="0 0 0"/>
+      <parent link="${prefix}link6"/>
+      <child link="${prefix}gripper"/>
+    </joint>
     <!-- Camera frame -->
     <link name="${prefix}camera"/>
@@ -218,4 +225,11 @@
       <child link="${prefix}camera"/>
     </joint>
+    <!-- Aruco -->
+<!--     <link name="${prefix}aruco"/>
+    <joint name="${prefix}base-aruco" type="fixed">
+      <origin xyz="-0.035 -0.214 0.353" rpy="${radians(-106.984)} ${radians(-23.960)} ${radians(-172.926)}"/>
+      <parent link="${prefix}base_link"/>
+      <child link="${prefix}aruco"/>
+    </joint> -->
   </xacro:macro>
 </robot>
