Commit message: added gripper control to ros2-control

File: mycobot_320_description/urdf/mycobot_320.ros2_control.xacro (robot description, xacro)
@@ -94,4 +94,15 @@
         <!-- <state_interface name="velocity"/> -->
       </joint>
+      <joint name="${prefix}gripper">
+        <command_interface name="position">
+          <param name="min">-3.14</param>
+          <param name="max">3.14</param>
+        </command_interface>
+        <state_interface name="position">
+          <!-- Initial position for the GenericSystem and simulation -->
+          <param name="initial_value">0</param>
+        </state_interface>
+        <!-- <state_interface name="velocity"/> -->
+      </joint>
     </ros2_control>
   </xacro:macro>

File: mycobot_320_description/urdf/mycobot_320.srdf.xacro (robot description, xacro)
@@ -8,5 +8,9 @@
         <joint name="joint5" />
         <joint name="joint6" />
+        <joint name="gripper" />
     </group>
+<!--     <group name="gripper_group">
+        <joint name="gripper" />
+    </group> -->
     <group_state name="init_pose" group="arm_group">
         <joint name="joint1" value="0" />

File: mycobot_320_description/urdf/mycobot_320_macro.xacro (robot description, xacro)
@@ -203,4 +203,14 @@
       <dynamics damping="0" friction="0"/>
     </joint>
+    <link name="${prefix}gripper_link"/>
+    <joint name="${prefix}gripper" type="revolute">
+      <parent link="${prefix}link6" />
+      <child link="${prefix}gripper_link" />
+      <origin xyz="0 0 0" rpy="0 0 0" />
+      <axis xyz="0 0 1" />
+      <limit lower="-3.14" upper="3.14"
+             effort="${joint6_effort_limit}" velocity="${joint6_velocity_limit}"/>
+      <dynamics damping="0" friction="0"/>
+    </joint>
     <!-- ROS-Industrial 'tool0' frame - all-zeros tool frame -->
     <link name="${prefix}tool0"/>

Commit message: wip

File: mycobot_320_description/urdf/mycobot_320.ros2_control.xacro (robot description, xacro)
@@ -94,5 +94,28 @@
         <!-- <state_interface name="velocity"/> -->
       </joint>
+     <joint name="gripper_controller">
+       <command_interface name="position">
+         <param name="min">0</param>
+         <param name="max">50</param>
+       </command_interface>
+            <state_interface name="position">
+              <param name="initial_value">0</param>
+            </state_interface>
+     </joint>
     </ros2_control>
+<!-- <ros2_control name="ElectricGripper" type="system">
+ <hardware>
+   <plugin>mock_components/GenericSystem</plugin>
+ </hardware>
+ <joint name="gripper_controller">
+   <command_interface name="position">
+     <param name="min">0</param>
+     <param name="max">50</param>
+   </command_interface>
+        <state_interface name="position">
+          <param name="initial_value">0</param>
+        </state_interface>
+ </joint>
+</ros2_control> -->
   </xacro:macro>
 </robot>

Commit message: working with fake hardware

File: mycobot_320_description/urdf/mycobot_320.ros2_control.xacro (robot description, xacro)
@@ -96,6 +96,6 @@
      <joint name="gripper_controller">
        <command_interface name="position">
-         <param name="min">0</param>
-         <param name="max">50</param>
+         <param name="min">-100</param>
+         <param name="max">100</param>
        </command_interface>
             <state_interface name="position">
@@ -104,18 +104,4 @@
      </joint>
     </ros2_control>
-<!-- <ros2_control name="ElectricGripper" type="system">
- <hardware>
-   <plugin>mock_components/GenericSystem</plugin>
- </hardware>
- <joint name="gripper_controller">
-   <command_interface name="position">
-     <param name="min">0</param>
-     <param name="max">50</param>
-   </command_interface>
-        <state_interface name="position">
-          <param name="initial_value">0</param>
-        </state_interface>
- </joint>
-</ros2_control> -->
   </xacro:macro>
 </robot>
